Commit message: Update README.md and add scripts

File: urdf/gazebo.urdf.xacro (robot description, xacro)
@@ -74,9 +74,9 @@
     </gazebo>
     <!-- RL leg -->
-    <gazebo reference="LR_hip">
+    <gazebo reference="RL_hip">
         <mu1>0.2</mu1>
         <mu2>0.2</mu2>
     </gazebo>
-    <gazebo reference="LR_upper_leg_link">
+    <gazebo reference="RL_upper_leg_link">
         <mu1>0.2</mu1>
         <mu2>0.2</mu2>
@@ -85,10 +85,10 @@
         <kd>1.0</kd>
     </gazebo>
-    <gazebo reference="LR_lower_leg_link">
+    <gazebo reference="RL_lower_leg_link">
         <mu1>0.2</mu1>
         <mu2>0.2</mu2>
         <self_collide>1</self_collide>
     </gazebo>
-    <gazebo reference="LR_foot_link">
+    <gazebo reference="RL_foot_link">
         <mu1>0.6</mu1>
         <mu2>0.6</mu2>

File: urdf/go2_description.urdf.xacro (robot description, xacro)
@@ -109,7 +109,7 @@
     <axis xyz="0 0 0" />
   </joint>
-  <xacro:go2_leg name="LF" x_joint="0.1934" y_joint="0.0465" y_thigh_joint="0.0955"/>
-  <xacro:go2_leg name="RF" x_joint="0.1934" y_joint="-0.0465" y_thigh_joint="-0.0955"/>
-  <xacro:go2_leg name="LR" x_joint="-0.1934" y_joint="0.0465" y_thigh_joint="0.0955"/>
+  <xacro:go2_leg name="FL" x_joint="0.1934" y_joint="0.0465" y_thigh_joint="0.0955"/>
+  <xacro:go2_leg name="FR" x_joint="0.1934" y_joint="-0.0465" y_thigh_joint="-0.0955"/>
+  <xacro:go2_leg name="RL" x_joint="-0.1934" y_joint="0.0465" y_thigh_joint="0.0955"/>
   <xacro:go2_leg name="RR" x_joint="-0.1934" y_joint="-0.0465" y_thigh_joint="-0.0955"/>
   <xacro:include filename="$(find go2_description)/urdf/gazebo.urdf.xacro"/>

File: urdf/leg.urdf.xacro (robot description, xacro)
@@ -3,17 +3,17 @@
   <xacro:macro name="go2_leg" params="name  x_joint y_joint y_thigh_joint" >
     <!-- <xacro:include filename="$(find go2_description)/urdf/transmission.urdf.xacro"/> -->
-    <xacro:property name="LF" value="LF" />
-    <xacro:property name="RF" value="RF" />
-    <xacro:property name="LR" value="LR" />
+    <xacro:property name="FL" value="FL" />
+    <xacro:property name="FR" value="FR" />
+    <xacro:property name="RL" value="RL" />
     <xacro:property name="RR" value="RR" />
     <link name="${name}_hip">
       <inertial>
-        <xacro:if value="${(name == LF)}">
+        <xacro:if value="${(name == FL)}">
           <origin xyz="-0.0054 0.00194 -0.000105" rpy="0 0 0" />
         </xacro:if>
-        <xacro:if value="${(name == RF)}">
+        <xacro:if value="${(name == FR)}">
           <origin xyz="-0.0054 -0.00194 -0.000105" rpy="0 0 0" />
         </xacro:if>
-        <xacro:if value="${(name == LR)}">
+        <xacro:if value="${(name == RL)}">
           <origin xyz="0.0054 0.00194 -0.000105" rpy="0 0 0" />
         </xacro:if>
@@ -62,8 +62,8 @@
         <origin xyz="0 0 0" rpy="0 0 0" />
         <geometry>
-          <xacro:if value="${(name == LF) or (name == LR)}">
+          <xacro:if value="${(name == FL) or (name == RL)}">
             <mesh filename="file://$(find go2_description)/dae/thigh.dae" scale="1 1 1"/>
           </xacro:if>
-           <xacro:if value="${(name == RF) or (name == RR)}">
+           <xacro:if value="${(name == FR) or (name == RR)}">
             <mesh filename="file://$(find go2_description)/dae/thigh_mirror.dae" scale="1 1 1"/>
           </xacro:if>
@@ -81,5 +81,5 @@
       </collision>
     </link>
-    <joint name="${name}_upper_leg_joint" type="revolute">
+    <joint name="${name}_thigh_joint" type="revolute">
       <origin xyz="0 ${y_thigh_joint} 0" rpy="0 0 0" />
       <parent link="${name}_hip" />
@@ -100,8 +100,8 @@
         <origin xyz="0 0 0" rpy="0 0 0" />
         <geometry>
-          <xacro:if value="${(name == LF) or (name == LR)}">
+          <xacro:if value="${(name == FL) or (name == RL)}">
             <mesh filename="file://$(find go2_description)/dae/calf.dae" scale="1 1 1"/>
           </xacro:if>
-           <xacro:if value="${(name == RF) or (name == RR)}">
+           <xacro:if value="${(name == FR) or (name == RR)}">
             <mesh filename="file://$(find go2_description)/dae/calf_mirror.dae" scale="1 1 1"/>
           </xacro:if>
@@ -119,5 +119,5 @@
       </collision>
     </link>
-    <joint name="${name}_lower_leg_joint" type="revolute">
+    <joint name="${name}_calf_joint" type="revolute">
       <origin xyz="0 0 -0.213" rpy="0 0 0" />
       <parent link="${name}_thigh" />
@@ -166,10 +166,10 @@
         <state_interface name="velocity"/>
       </joint>
-      <joint name="${name}_upper_leg_joint">
+      <joint name="${name}_thigh_joint">
         <command_interface name="effort"/>
         <state_interface name="position"/>
         <state_interface name="velocity"/>
       </joint>
-      <joint name="${name}_lower_leg_joint">
+      <joint name="${name}_calf_joint">
         <command_interface name="effort"/>
         <state_interface name="position"/>

File: urdf/transmission.urdf.xacro (robot description, xacro)
@@ -14,5 +14,5 @@
         <transmission name="${name}_upper_leg_tran">
             <type>transmission_interface/SimpleTransmission</type>
-            <joint name="${name}_upper_leg_joint">
+            <joint name="${name}_thigh_joint">
             <hardwareInterface>hardware_interface/EffortJointInterface</hardwareInterface>
             </joint>
@@ -24,5 +24,5 @@
         <transmission name="${name}_lower_leg_tran">
             <type>transmission_interface/SimpleTransmission</type>
-            <joint name="${name}_lower_leg_joint">
+            <joint name="${name}_calf_joint">
             <hardwareInterface>hardware_interface/EffortJointInterface</hardwareInterface>
             </joint>
